File: pcb/forgepad.kicad_pcb (KiCad board)
At the start: 2 copper layers, 67.2 x 93.2 mm, 13 parts, among them SW1 SW_Push, SW2 SW_Push, SW3 SW_Push, SW4 SW_Push, SW5 SW_Push, SW6 SW_Push, SW7 SW_Push, SW8 SW_Push, SW9 SW_Push, U1 XIAO-RP2040-DIP

Commit message: Update forgepad.kicad_pcb
Parts:
- D2: value SK6812 -> SK6812MINI-E
Changed lines of the file:
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@@
 			)
 		)
-		(property "Value" "SK6812"
-			(at 0 3.25 0)
-			(layer "F.Fab")
+		(property "Value" "SK6812MINI-E"
+			(at 1.27 -5.715 0)
 			(effects
 				(font
-					(size 1 1)
-					(thickness 0.15)
+					(size 1.27 1.27)
+					(thickness 0.254)
+					(bold yes)
 				)
+				(justify left top)
 			)
 		)
@@
 			)
 		)
-		(property "Description" ""
+		(property "Description" "RGB LED with integrated controller"
 			(at 0 0 0)
-			(unlocked yes)
-			(layer "F.Fab")
-			(hide yes)
 			(effects
 				(font
 					(size 1.27 1.27)
-					(thickness 0.15)
 				)
+				(hide yes)
 			)
 		)
